File: DeltaCore/hamilton.brd (EAGLE design)
At the start: 45 x 41.5 mm, 70 parts, among them Q3 MOSFET-NCHANNEL_SOT23-3, Q4 MOSFET-NCHANNEL_SOT23-3, Q5 MOSFET-NCHANNEL_SOT23-3, Q6 MOSFET-NCHANNEL_SOT23-3, Q7 NFET_AON7408, Q8 NFET_AON7408, U1 SAMR21, U10 PCA9557, U3 MMA7660FC, U4 AT30TS74, U5 MCP73871-2AAI/ML, U7 BQ29718, U8 MCP1824ST-3302E/DB, U9 TPS61090, X1 XTAL

Commit message: latest updates
Routing:
- net LBO: track 43.4 -> 44.2 mm, vias 0 -> 1
- net GND: vias 58 -> 59
Other:
- board text added: "+"
- board text added: "+3V3"
- board text added: "+5V"
- board text added: "-"
- board text added: "BAT"
- board text added: "CHRG"
- board text added: "DC"
- board text added: "LBO"
Changed lines of the file:
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@@
 <layers>
 <layer number="1" name="Top" color="4" fill="1" visible="yes" active="yes"/>
-<layer number="2" name="Route2" color="1" fill="3" visible="no" active="yes"/>
+<layer number="2" name="Route2" color="1" fill="3" visible="yes" active="yes"/>
 <layer number="3" name="Route3" color="4" fill="3" visible="no" active="no"/>
 <layer number="14" name="Route14" color="1" fill="6" visible="no" active="no"/>
@@
 <layer number="27" name="tValues" color="7" fill="1" visible="no" active="yes"/>
 <layer number="28" name="bValues" color="7" fill="1" visible="no" active="yes"/>
-<layer number="29" name="tStop" color="7" fill="3" visible="no" active="yes"/>
+<layer number="29" name="tStop" color="7" fill="3" visible="yes" active="yes"/>
 <layer number="30" name="bStop" color="7" fill="6" visible="no" active="yes"/>
 <layer number="31" name="tCream" color="7" fill="4" visible="no" active="yes"/>
@@
 <text x="9.5758" y="20.2438" size="0.8128" layer="25" rot="R90">Q7</text>
 <text x="11.8364" y="13.843" size="0.8128" layer="25" rot="R180">Q8</text>
+<text x="9.398" y="11.049" size="0.8128" layer="25">CHRG</text>
+<text x="39.243" y="15.875" size="0.8128" layer="25">+3V3</text>
+<text x="20.447" y="17.145" size="0.8128" layer="25">+5V</text>
+<text x="24.638" y="20.447" size="0.8128" layer="25">LBO</text>
+<text x="3.556" y="7.747" size="0.8128" layer="25">5V</text>
+<text x="4.064" y="4.826" size="0.8128" layer="25">GND</text>
+<text x="3.937" y="2.413" size="0.8128" layer="25">DC</text>
+<text x="39.751" y="0.381" size="0.8128" layer="25">BAT</text>
+<text x="44.069" y="0.762" size="0.8128" layer="25">-</text>
+<text x="44.196" y="5.588" size="0.8128" layer="25">+</text>
+<circle x="10.668" y="10.033" radius="0.179603125" width="0.3048" layer="25"/>
 </plain>
 <attributes>
@@
 <attribute name="VALUE" x="25.7594" y="40.8526" size="1.27" layer="27" rot="R180"/>
 </element>
-<element name="JP2" library="pinhead" package="1X02" value="insole1" x="13.33464375" y="37.7859125" rot="R68.5"/>
-<element name="JP3" library="pinhead" package="1X02" value="insole2" x="11.47281875" y="33.059390625" rot="R68.5"/>
-<element name="JP4" library="pinhead" package="1X02" value="insole3" x="9.610990625" y="28.33286875" rot="R68.5"/>
-<element name="JP5" library="pinhead" package="1X02" value="insole4" x="7.749165625" y="23.606346875" rot="R68.5"/>
-<element name="JP6" library="pinhead" package="1X02" value="insole/wrist" x="5.8873375" y="18.879828125" rot="R68.5"/>
-<element name="JP7" library="pinhead" package="1X03" value="insole/fan/pwm" x="3.56005625" y="12.971675" rot="R68.5"/>
+<element name="JP2" library="pinhead" package="1X02" value="insole1" x="13.33464375" y="37.7859125" smashed="yes" rot="R68.5">
+<attribute name="NAME" x="15.627253125" y="35.133009375" size="1.27" layer="26" ratio="10" rot="R68.5"/>
+<attribute name="VALUE" x="15.35780625" y="34.259009375" size="1.27" layer="27" rot="R68.5"/>
+</element>
+<element name="JP3" library="pinhead" package="1X02" value="insole2" x="11.47281875" y="33.059390625" smashed="yes" rot="R68.5">
+<attribute name="NAME" x="14.019428125" y="30.6604875" size="1.27" layer="26" ratio="10" rot="R68.5"/>
+<attribute name="VALUE" x="13.49598125" y="29.5324875" size="1.27" layer="27" rot="R68.5"/>
+</element>
+<element name="JP4" library="pinhead" package="1X02" value="insole3" x="9.610990625" y="28.33286875" smashed="yes" rot="R68.5">
+<attribute name="NAME" x="11.9036" y="25.552965625" size="1.27" layer="26" ratio="10" rot="R68.5"/>
+<attribute name="VALUE" x="11.634153125" y="24.805965625" size="1.27" layer="27" rot="R68.5"/>
+</element>
+<element name="JP5" library="pinhead" package="1X02" value="insole4" x="7.749165625" y="23.606346875" smashed="yes" rot="R68.5">
+<attribute name="NAME" x="9.914775" y="20.82644375" size="1.27" layer="26" ratio="10" rot="R68.5"/>
+<attribute name="VALUE" x="9.772328125" y="20.07944375" size="1.27" layer="27" rot="R68.5"/>
+</element>
+<element name="JP6" library="pinhead" package="1X02" value="insole/wrist" x="5.8873375" y="18.879828125" smashed="yes" rot="R68.5">
+<attribute name="NAME" x="8.052946875" y="16.226925" size="1.27" layer="26" ratio="10" rot="R68.5"/>
+<attribute name="VALUE" x="7.9105" y="15.352925" size="1.27" layer="27" rot="R68.5"/>
+</element>
+<element name="JP7" library="pinhead" package="1X03" value="insole/fan/pwm" x="3.56005625" y="12.971675" smashed="yes" rot="R68.5">
+<attribute name="NAME" x="5.260209375" y="9.391140625" size="1.27" layer="26" ratio="10" rot="R68.5"/>
+<attribute name="VALUE" x="5.117759375" y="8.263140625" size="1.27" layer="27" rot="R68.5"/>
+</element>
 <element name="Q7" library="fets" package="VDFN3X38L" value="NFET_AON7408" x="11.176" y="20.066" smashed="yes"/>
 <element name="Q8" library="fets" package="VDFN3X38L" value="NFET_AON7408" x="10.16" y="15.494" smashed="yes" rot="R270"/>
-<element name="JP8" library="pinhead" package="1X03" value="PRU input" x="2.27" y="4.556" rot="R90"/>
+<element name="JP8" library="pinhead" package="1X03" value="PRU input" x="2.27" y="4.556" smashed="yes" rot="R90">
+<attribute name="NAME" x="5.7752" y="1.0508" size="1.27" layer="26" ratio="10" rot="R90"/>
+<attribute name="VALUE" x="5.445" y="0.746" size="1.27" layer="27" rot="R90"/>
+</element>
 <element name="U5" library="Microchip_By_element14_Batch_1" package="QFN50P400X400X100-21N" value="MCP73871-2AAI/ML" x="13.366" y="7.608" smashed="yes">
 <attribute name="OC_FARNELL" value="1642487" x="13.366" y="7.608" size="1.778" layer="27" display="off"/>
@@
 <wire x1="24.304" y1="1.186" x2="24.304" y2="1.18" width="0.1524" layer="1"/>
 <wire x1="24.304" y1="1.18" x2="25.908" y2="1.18" width="0.3048" layer="1"/>
-<wire x1="25.908" y1="1.18" x2="25.908" y2="2.92" width="0.3048" layer="1"/>
-<wire x1="27.532" y1="2.92" x2="25.908" y2="2.92" width="0.3048" layer="1"/>
 <wire x1="3.54" y1="4.556" x2="5.57" y2="4.556" width="0.3048" layer="1"/>
 <wire x1="5.57" y1="4.556" x2="5.57" y2="6.944" width="0.3048" layer="1"/>
@@
 <wire x1="25.4" y1="11.1252" x2="25.4" y2="12.8016" width="0.1524" layer="1"/>
 <wire x1="25.4" y1="12.8016" x2="25.5778" y2="12.8016" width="0.1524" layer="1"/>
+<wire x1="25.908" y1="1.18" x2="25.908" y2="2.921" width="0.3048" layer="1"/>
+<via x="25.908" y="2.921" extent="1-16" drill="0.3048"/>
+<wire x1="27.532" y1="2.92" x2="27.532" y2="2.921" width="0.3048" layer="1"/>
+<wire x1="27.532" y1="2.921" x2="25.908" y2="2.921" width="0.3048" layer="1"/>
 </signal>
 <signal name="N$3">
@@
 <wire x1="42.672" y1="16.1544" x2="42.672" y2="17.272" width="0.3048" layer="1"/>
 <wire x1="42.672" y1="17.272" x2="42.037" y2="17.272" width="0.3048" layer="1"/>
-<via x="42.037" y="17.272" extent="1-16" drill="0.3048"/>
+<via x="42.037" y="17.272" extent="1-16" drill="0.3048" alwaysstop="yes"/>
 <wire x1="42.672" y1="17.272" x2="42.799" y2="17.272" width="0.3048" layer="1"/>
 <wire x1="42.799" y1="17.272" x2="42.799" y2="18.542" width="0.3048" layer="1"/>
@@
 <wire x1="21.8182" y1="40.8432" x2="25.4" y2="40.8432" width="0.1524" layer="1"/>
 <wire x1="25.4" y1="40.386" x2="25.4" y2="40.8432" width="0.1524" layer="1"/>
-<via x="25.4" y="40.386" extent="1-16" drill="0.3048"/>
+<via x="25.4" y="40.386" extent="1-16" drill="0.3048" alwaysstop="yes"/>
 <wire x1="31.242" y1="40.8432" x2="25.4" y2="40.8432" width="0.1524" layer="1"/>
 <wire x1="31.242" y1="40.8432" x2="31.242" y2="38.989" width="0.1524" layer="1"/>
@@
 <wire x1="26.543" y1="40.259" x2="26.543" y2="39.751" width="0.1524" layer="1"/>
 <wire x1="26.543" y1="39.751" x2="29.464" y2="39.751" width="0.1524" layer="1"/>
-<via x="26.543" y="40.259" extent="1-16" drill="0.3048"/>
+<via x="26.543" y="40.259" extent="1-16" drill="0.3048" alwaysstop="yes"/>
 <wire x1="29.464" y1="37.588" x2="29.464" y2="39.751" width="0.1524" layer="1"/>
 <wire x1="29.464" y1="37.588" x2="36.8808" y2="37.588" width="0.1524" layer="1"/>
@@
 <wire x1="31.115" y1="7.874" x2="31.115" y2="7.913" width="0.1524" layer="1"/>
 <wire x1="28.448" y1="8.551" x2="28.448" y2="8.001" width="0.3048" layer="1"/>
-<via x="28.448" y="7.112" extent="1-16" drill="0.3048"/>
+<via x="28.448" y="7.112" extent="1-16" drill="0.3048" alwaysstop="yes"/>
 <wire x1="28.448" y1="7.913" x2="28.448" y2="7.112" width="0.3048" layer="1"/>
 <wire x1="31.115" y1="7.913" x2="28.448" y2="7.913" width="0.3048" layer="1"/>
@@
 <wire x1="18.669" y1="12.827" x2="21.844" y2="16.002" width="0.3048" layer="16"/>
 <wire x1="21.844" y1="16.002" x2="21.844" y2="16.51" width="0.3048" layer="16"/>
-<via x="21.844" y="16.51" extent="1-16" drill="0.3048"/>
+<via x="21.844" y="16.51" extent="1-16" drill="0.3048" alwaysstop="yes"/>
 <wire x1="21.844" y1="16.51" x2="21.844" y2="14.492" width="0.3048" layer="1"/>
 <wire x1="26.797" y1="15.875" x2="26.797" y2="16.51" width="0.3048" layer="1"/>
@@
 <wire x1="28.194" y1="16.6624" x2="28.194" y2="17.272" width="0.1524" layer="1"/>
 <wire x1="28.194" y1="17.272" x2="26.3906" y2="17.272" width="0.1524" layer="1"/>
-<wire x1="26.3906" y1="17.272" x2="26.3906" y2="21.209" width="0.1524" layer="1"/>
-<wire x1="26.3906" y1="21.209" x2="27.686" y2="21.209" width="0.1524" layer="1"/>
 <wire x1="27.686" y1="21.209" x2="27.686" y2="32.893" width="0.1524" layer="1"/>
 <wire x1="27.686" y1="32.893" x2="31.2166" y2="32.893" width="0.1524" layer="1"/>
@@
 <wire x1="35.56" y1="36.6268" x2="35.56" y2="37.211" width="0.1524" layer="1"/>
 <wire x1="35.56" y1="37.211" x2="35.5854" y2="37.211" width="0.1524" layer="1"/>
+<wire x1="26.3906" y1="17.272" x2="26.3906" y2="19.939" width="0.1524" layer="1"/>
+<wire x1="26.3906" y1="19.939" x2="25.654" y2="19.939" width="0.1524" layer="1"/>
+<wire x1="26.3906" y1="19.939" x2="26.416" y2="19.939" width="0.1524" layer="1"/>
+<wire x1="26.416" y1="19.939" x2="26.416" y2="21.209" width="0.1524" layer="1"/>
+<wire x1="26.416" y1="21.209" x2="27.686" y2="21.209" width="0.1524" layer="1"/>
+<via x="25.654" y="19.939" extent="1-16" drill="0.3048" alwaysstop="yes"/>
 </signal>
 <signal name="N$27">

Commit message: next version
Parts:
- removed JP4: insole3, pinhead:1X02
- removed JP5: insole4, pinhead:1X02
- removed JP6: insole/wrist, pinhead:1X02
- removed JP7: insole/fan/pwm, pinhead:1X03
- removed JP9: (no value), pinhead:1X01
- removed R12: 10k, resistor:R0402
- added R20, R21, R22, R23, R24, R25: 10k, resistor:R0402
- JP2: value insole1 -> (none); device pinhead:1X02 -> pinhead:1X07
- JP3: value insole2 -> (none); device pinhead:1X02 -> pinhead:1X04
- moved Q5 26.0 mm to (8.70, 41.5), turned to 90 degrees
- moved Q6 22.4 mm to (8.70, 37.8), turned to 90 degrees
- moved Q8 18.9 mm to (18.4, 32.5), turned to 90 degrees
- moved Q3 14.7 mm to (8.60, 48.8), turned to 90 degrees
- moved Q4 14.5 mm to (8.62, 45.0), turned to 90 degrees
- moved Q7 14.2 mm to (8.46, 34.0), turned to 90 degrees
- moved JP3 11.4 mm to (3.00, 25.5), turned to 270 degrees
- moved JP2 11.2 mm to (3.00, 42.0), turned to 270 degrees
- moved C14 10.8 mm to (8.92, 18.0), turned to 0 degrees
- moved R14 8.26 mm to (21.4, 46.3)
- moved U10 8.26 mm to (19.1, 41.8)
- moved C11 8.17 mm to (29.4, 43.8)
- moved JP8 8.03 mm to (2.98, 12.6)
- moved RT1 6.69 mm to (12.4, 17.7)
- moved R18 5.63 mm to (20.5, 5.46)
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Connections:
- removed net EN: R12.2, U1.25, U9.EN
- removed net N$39: JP7.2, Q8.1, Q8.2, Q8.3
- removed net N$8: JP9.1, R3.2
- new net ADC7: JP3.4, R3.2
- new net D27: JP3.2, U1.25
- new net D28: JP3.3, U1.27
- new net N$11: JP2.5, Q7.5, Q7.6, Q7.7, Q7.8, Q7.PAD
- new net N$26: JP2.6, Q8.5, Q8.6, Q8.7, Q8.8, Q8.PAD
- net 5V: now also JP2.7; no longer JP2.1, JP3.1, JP4.1, JP5.1, JP6.1, JP7.1
- net D25: now also JP3.1; no longer JP7.3
- net GND: now also Q3.2, Q4.2, Q5.2, Q6.2, Q7.1, Q7.2, Q7.3, Q8.1, Q8.2, Q8.3, R20.1, R21.1, R22.1, R23.1, R24.1, R25.1; no longer Q3.3, Q4.3, Q5.3, Q6.3, Q7.5, Q7.6, Q7.7, Q7.8, Q7.PAD, Q8.5, Q8.6, Q8.7, Q8.8, Q8.PAD, R12.1
- net N$14: now also JP2.1, Q3.3; no longer JP2.2, Q3.2
- net N$20: no longer C15.1, JP1.1, R18.1, R8.2, U5.14, U5.15, U5.16
- net N$30: now also R25.2
- net N$31: now also R20.2
- net N$32: now also R21.2
- net N$33: now also R22.2
- net N$34: now also JP2.2, Q4.3; no longer JP3.2, Q4.2
- net N$35: now also JP2.3, Q5.3; no longer JP4.2, Q5.2
- net N$36: now also JP2.4, Q6.3; no longer JP5.2, Q6.2
- net N$37: now also C15.1, JP1.1, R18.1, R8.2, U5.14, U5.15, U5.16; no longer JP6.2, Q7.1, Q7.2, Q7.3
- net N$40: now also R23.2
- net N$41: now also R24.2
- net OUT: now also U9.EN
Routing:
- net N$37: track 8.72 -> 47.6 mm
- net N$20: track 50.4 -> 13.4 mm
- net D28: track 0.00 -> 29.9 mm, vias 0 -> 1
- net EN: track 29.9 -> 0.00 mm, vias 2 -> 0
- net N$8: track 29.3 -> 0.00 mm, vias 1 -> 0
- net D27: track 0.00 -> 28.6 mm, vias 0 -> 1
- net ADC7: track 0.00 -> 28.6 mm, vias 0 -> 1
- net N$41: track 38.6 -> 16.2 mm, vias 2 -> 0
- net GND: track 248.7 -> 226.6 mm, vias 59 -> 64
- net N$26: track 0.00 -> 21.1 mm, vias 0 -> 1
- net D25: track 46.2 -> 29.3 mm
- net SCL: track 55.7 -> 68.6 mm
- net N$11: track 0.00 -> 12.2 mm
- net N$31: track 8.03 -> 19.4 mm
- net N$30: track 8.14 -> 19.2 mm
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- removed copper zone on layer 15, net 5V
Other:
- board size 45 x 41.5 mm -> 40 x 52 mm
- board text added: "10/24/16"
- board text added: "V+"
- board text removed: "5V"
- board text removed: "CHRG"
- board text removed: "D25"
- board text removed: "DC"
- board text removed: "Q7"
- board text removed: "Q8"

Commit message: update
Parts:
- R15: value ?? -> 523k
- R4: value ?? -> 110k
Changed lines of the file:
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@@
 <attribute name="VALUE" x="5.4494" y="3.5074" size="1.016" layer="27" ratio="10" rot="SR0"/>
 </element>
-<element name="R4" library="resistor" package="R0603" value="??" x="1.858" y="1.905" smashed="yes" rot="R90">
+<element name="R4" library="resistor" package="R0603" value="110k" x="1.858" y="1.905" smashed="yes" rot="R90">
 <attribute name="NAME" x="1.1468" y="0.4064" size="0.8128" layer="25" rot="R90"/>
 <attribute name="VALUE" x="3.763" y="1.27" size="1.27" layer="27" rot="R90"/>
 </element>
-<element name="R15" library="resistor" package="R0603" value="??" x="5.033" y="1.905" smashed="yes" rot="R270">
+<element name="R15" library="resistor" package="R0603" value="523k" x="5.033" y="1.905" smashed="yes" rot="R270">
 <attribute name="NAME" x="6.6078" y="0.381" size="0.8128" layer="25" rot="R90"/>
 <attribute name="VALUE" x="3.128" y="2.54" size="1.27" layer="27" rot="R270"/>
@@
 <vertex x="32.084" y="51.894"/>
 <vertex x="32.338" y="20.828"/>
-<vertex x="44.958" y="20.828"/>
-<vertex x="44.958" y="7.62"/>
+<vertex x="40.132" y="20.828"/>
+<vertex x="40.132" y="7.62"/>
 <vertex x="29.21" y="7.112"/>
 <vertex x="29.21" y="4.064"/>
@@
 <vertex x="32.338" y="51.816"/>
 <vertex x="32.338" y="20.574"/>
-<vertex x="44.958" y="20.828"/>
-<vertex x="45.212" y="7.62"/>
+<vertex x="39.878" y="20.828"/>
+<vertex x="40.132" y="7.62"/>
 <vertex x="29.464" y="7.366"/>
 <vertex x="29.464" y="3.81"/>
