File: DeltaCore/hamilton.sch (EAGLE design)
At the start: 69 parts, among them Q1 CSD16301Q2, Q2 CSD16301Q2, Q3 MOSFET-NCHANNEL_SOT23-3, Q4 MOSFET-NCHANNEL_SOT23-3, Q5 MOSFET-NCHANNEL_SOT23-3, Q6 MOSFET-NCHANNEL_SOT23-3, Q7 NFET_AON7408, Q8 NFET_AON7408, U1 SAMR21, U10 PCA9557, U3 MMA7660FC, U4 AT30TS74, U5 MCP73871-2AAI/ML, U7 BQ29718, U8 MCP1824ST-3302E/DB, U9 TPS61090, X1 XTAL

Commit message: fixes
Parts:
- removed C13, C7: 100nF, storm:0603_CAPACITOR0402
- added R17: 2k, resistor:R-US_R0402
- added R18: 13k, resistor:R-US_R0402
- added R19: 5k, resistor:R-US_R0402
- R12: value 1.6k -> 10k; device resistor:R-US_R0603 -> resistor:R-US_R0402
- R13: value 1.6k -> 68k; device resistor:R-US_R0603 -> resistor:R-US_R0402
- R14: value 1.1k -> 10k
Connections:
- removed net N$29: R14.1, U10.RESET
- new net BAT: R18.2, R19.1, U1.PA08
- new net EN: R12.2, U1.PA27, U9.EN
- new net N$12: U1.PA09
- new net N$15: U1.PA14
- new net N$17: U1.PA15
- new net N$42: U1.PA24
- new net RST: R14.1, U1.PA18, U10.RESET
- new net WIT: R13.1, R17.2, U1.PA06
- net +3V3: no longer C13.P$1, C7.P$1, R12.2, R13.2, R14.2
- net ACC: no longer U1.PA06
- net GND: now also R12.1, R14.2, R17.1, R19.2; no longer C13.P$2, C7.P$2
- net LBO: now also U1.PA19
- net N$1: now also JP8.1, R13.2, R4.2; no longer R15.2, R4.1, U5.VPCC
- net N$20: now also R18.1
- net RECT: now also R15.2, R4.1, U5.VPCC; no longer JP8.1, R4.2
- net SCL: no longer R12.1
- net SDA: no longer R13.1
Other:
- moved on the sheet: R12, R13

Commit message: more
Parts:
- renumbered U$2 to RT1
Connections:
- removed net ACC: U3.!INT!
- removed net OOB: U$1.TDO/SWO
- removed net SD: U1.PA28
Changed lines of the file:
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@@
 <part name="R6" library="resistor" deviceset="R-US_" device="R0603" value="2k"/>
 <part name="C15" library="resistor" deviceset="C-EU" device="C0603" value="4.7uF"/>
-<part name="U$2" library="varistor" deviceset="NCP15XH103J03RC" device=""/>
+<part name="RT1" library="varistor" deviceset="NCP15XH103J03RC" device=""/>
 <part name="R7" library="resistor" deviceset="R-US_" device="R0603" value="2.2k"/>
 <part name="Q1" library="insole" deviceset="CSD16301Q2" device="" value=""/>
@@
 <instance part="R6" gate="G$1" x="-50.8" y="-45.72" rot="R90"/>
 <instance part="C15" gate="G$1" x="-30.48" y="-45.72"/>
-<instance part="U$2" gate="G$1" x="-45.72" y="-35.56"/>
+<instance part="RT1" gate="G$1" x="-45.72" y="-35.56"/>
 <instance part="R7" gate="G$1" x="-17.78" y="-45.72" rot="R90"/>
 <instance part="Q1" gate="G$1" x="-5.08" y="-50.8" rot="R270"/>
@@
 <wire x1="-50.8" y1="-53.34" x2="-50.8" y2="-50.8" width="0.1524" layer="91"/>
 <junction x="-58.42" y="-53.34"/>
-<pinref part="U$2" gate="G$1" pin="1"/>
+<pinref part="RT1" gate="G$1" pin="1"/>
 <wire x1="-40.64" y1="-35.56" x2="-38.1" y2="-35.56" width="0.1524" layer="91"/>
 <wire x1="-38.1" y1="-35.56" x2="-38.1" y2="-53.34" width="0.1524" layer="91"/>
@@
 </segment>
 </net>
-<net name="ACC" class="0">
-<segment>
-<pinref part="U3" gate="G$1" pin="!INT!"/>
-<wire x1="104.14" y1="33.02" x2="101.6" y2="33.02" width="0.1524" layer="91"/>
-<label x="101.6" y="33.02" size="1.27" layer="95" rot="R180" xref="yes"/>
-</segment>
-</net>
-<net name="SD" class="0">
-<segment>
-<pinref part="U1" gate="G$1" pin="PA28"/>
-<wire x1="73.66" y1="45.72" x2="76.2" y2="45.72" width="0.1524" layer="91"/>
-<label x="76.2" y="45.72" size="1.27" layer="95" xref="yes"/>
-</segment>
-</net>
 <net name="!RESET!" class="0">
 <segment>
@@
 <pinref part="C3" gate="G$1" pin="P$1"/>
 <wire x1="27.94" y1="48.26" x2="33.02" y2="48.26" width="0.1524" layer="91"/>
-</segment>
-</net>
-<net name="OOB" class="0">
-<segment>
-<pinref part="U$1" gate="G$1" pin="TDO/SWO"/>
-<wire x1="68.58" y1="78.74" x2="66.04" y2="78.74" width="0.1524" layer="91"/>
-<label x="66.04" y="78.74" size="1.27" layer="95" rot="R180" xref="yes"/>
 </segment>
 </net>
@@
 <net name="N$19" class="0">
 <segment>
-<pinref part="U$2" gate="G$1" pin="2"/>
+<pinref part="RT1" gate="G$1" pin="2"/>
 <wire x1="-71.12" y1="-35.56" x2="-50.8" y2="-35.56" width="0.1524" layer="91"/>
 <pinref part="U5" gate="A" pin="THERM"/>

Commit message: next version
Parts:
- removed JP4: insole3, pinhead:PINHD-1X2
- removed JP5: insole4, pinhead:PINHD-1X2
- removed JP6: insole/wrist, pinhead:PINHD-1X2
- removed JP7: insole/fan/pwm, pinhead:PINHD-1X3
- removed JP9: (no value), pinhead:PINHD-1X1
- removed R12: 10k, resistor:R-US_R0402
- added R20, R21, R22, R23, R24, R25: 10k, resistor:R-US_R0402
- JP2: value insole1 -> (none); device pinhead:PINHD-1X2 -> pinhead:PINHD-1X7
- JP3: value insole2 -> (none); device pinhead:PINHD-1X2 -> pinhead:PINHD-1X4
Connections:
- removed net EN: R12.2, U1.PA27, U9.EN
- removed net N$39: JP7.2, Q8.S@1, Q8.S@2, Q8.S@3
- removed net N$8: JP9.1, R3.2
- new net ADC7: JP3.4, R3.2
- new net D27: JP3.2, U1.PA27
- new net D28: JP3.3, U1.PA28
- new net N$11: JP2.5, Q7.D@1, Q7.D@2, Q7.D@3, Q7.D@4, Q7.D@5
- new net N$26: JP2.6, Q8.D@1, Q8.D@2, Q8.D@3, Q8.D@4, Q8.D@5
- net 5V: now also JP2.7; no longer JP2.1, JP3.1, JP4.1, JP5.1, JP6.1, JP7.1
- net D25: now also JP3.1; no longer JP7.3
- net GND: now also Q3.S, Q4.S, Q5.S, Q6.S, Q7.S@1, Q7.S@2, Q7.S@3, Q8.S@1, Q8.S@2, Q8.S@3, R20.1, R21.1, R22.1, R23.1, R24.1, R25.1; no longer Q3.D, Q4.D, Q5.D, Q6.D, Q7.D@1, Q7.D@2, Q7.D@3, Q7.D@4, Q7.D@5, Q8.D@1, Q8.D@2, Q8.D@3, Q8.D@4, Q8.D@5, R12.1
- net N$14: now also JP2.1, Q3.D; no longer JP2.2, Q3.S
- net N$20: no longer C15.1, JP1.1, R18.1, R8.2, U5.VBAT, U5.VBAT_2, U5.VBAT_SENSE
- net N$30: now also R25.2
- net N$31: now also R20.2
- net N$32: now also R21.2
- net N$33: now also R22.2
- net N$34: now also JP2.2, Q4.D; no longer JP3.2, Q4.S
- net N$35: now also JP2.3, Q5.D; no longer JP4.2, Q5.S
- net N$36: now also JP2.4, Q6.D; no longer JP5.2, Q6.S
- net N$37: now also C15.1, JP1.1, R18.1, R8.2, U5.VBAT, U5.VBAT_2, U5.VBAT_SENSE; no longer JP6.2, Q7.S@1, Q7.S@2, Q7.S@3
- net N$40: now also R23.2
- net N$41: now also R24.2
- net OUT: now also U9.EN

Commit message: update
Parts:
- R15: value ?? -> 523k
- R4: value ?? -> 110k
Changed lines of the file:
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@@
 <part name="JP8" library="pinhead" deviceset="PINHD-1X3" device="" value="PRU input"/>
 <part name="U5" library="Microchip_By_element14_Batch_1" deviceset="MCP73871-2AAI/ML" device=""/>
-<part name="R4" library="resistor" deviceset="R-US_" device="R0603" value="??"/>
-<part name="R15" library="resistor" deviceset="R-US_" device="R0603" value="??"/>
+<part name="R4" library="resistor" deviceset="R-US_" device="R0603" value="110k"/>
+<part name="R15" library="resistor" deviceset="R-US_" device="R0603" value="523k"/>
 <part name="R3" library="resistor" deviceset="R-US_" device="R0402" value="20k"/>
 <part name="R16" library="resistor" deviceset="R-US_" device="R0402" value="5k"/>
