File: DeltaCore2/hamilton.brd (EAGLE design)
At the start: 40 x 52 mm, 69 parts, among them Q3 MOSFET-NCHANNEL_SOT23-3, Q4 MOSFET-NCHANNEL_SOT23-3, Q5 MOSFET-NCHANNEL_SOT23-3, Q6 MOSFET-NCHANNEL_SOT23-3, Q7 NFET_AON7408, Q8 NFET_AON7408, U1 SAMR21, U10 PCA9557, U2 74LVC1T45, U3 MMA7660FC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

Commit message: update
Parts:
- added C7: 10uF, resistor:C0603
- added D1: IP4220CZ6, insole:SOT457
- added D2: CZRU52C4V7, insole:R0603
- added D3, D4: DB2G32600L1, insole:R0402
- added D5, D6: (no value), resistor:R0603
- added R11: 0, resistor:R0603
- added R26, R27: (no value), resistor:R0402
- R10: value 390k -> 75k
- R15: value 523k -> 110k
- R4: value 110k -> 523k
- R9: value 1.48M -> 374k
- moved C19 12.3 mm to (13.6, 18.3)
- moved C20 10.2 mm to (13.6, 20.1), turned to 180 degrees
- moved RT1 5.08 mm to (12.4, 12.6)
- moved R10 4.71 mm to (21.7, 7.07), turned to 0 degrees
- moved C14 4.57 mm to (8.92, 13.4)
Connections:
- new net LDOIN: C17.1, R11.1, U8.1
- new net N$38: D5.2, R26.1
- new net N$39: D6.2, R27.1
- net +3V3: now also D1.6
- net 5V: now also D4.C
- net ADC7: now also D1.5
- net D25: now also D1.1, D5.1
- net D27: now also D1.3, D6.1
- net D28: now also D1.4
- net GND: now also C7.2, D1.2, D2.A, R26.2, R27.2
- net N$25: now also D3.A
- net N$26: now also D4.A
- net N$37: now also D3.C
- net OUT: now also C7.1, R11.2; no longer C17.1, U8.1
- net RECT: now also D2.C
Routing:
- net D25: track 29.7 -> 101.8 mm, vias 1 -> 2
- net D27: track 27.0 -> 85.5 mm, vias 1 -> 3
- net OUT: track 70.3 -> 60.0 mm, vias 4 -> 2
- net D28: track 28.1 -> 37.7 mm, vias 1 -> 2
- net LDOIN: track 0.00 -> 9.35 mm
- net N$19: track 23.7 -> 18.7 mm
- net VCC: track 49.2 -> 44.6 mm
- net N$26: track 21.1 -> 23.9 mm
- net N$38: track 0.00 -> 2.21 mm
- net 5V: track 56.7 -> 58.8 mm
- net ADC7: track 31.5 -> 33.6 mm, vias 1 -> 2
- net N$39: track 0.00 -> 2.00 mm
- net GND: track 214.6 -> 212.6 mm, vias 62 -> 67
- net +3V3: track 42.6 -> 44.5 mm, vias 8 -> 9
- net N$28: track 10.2 -> 8.43 mm
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Other:
- board text added: "1"
- board text added: "2"
- board text added: "3"
- board text added: "4"
- board text added: "5"
- board text added: "5/11/17 v3"
- board text added: "6"
- board text added: "GT Fierro"
- board text removed: "10/24/16"
- board text removed: "G Fierro"
