File: DeltaCore2/hamilton.sch (EAGLE design)
At the start: 69 parts, among them Q1 CSD16301Q2, Q2 CSD16301Q2, Q3 MOSFET-NCHANNEL_SOT23-3, Q4 MOSFET-NCHANNEL_SOT23-3, Q5 MOSFET-NCHANNEL_SOT23-3, Q6 MOSFET-NCHANNEL_SOT23-3, Q7 NFET_AON7408, Q8 NFET_AON7408, U1 SAMR21, U10 PCA9557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

Commit message: update
Parts:
- added C7: 10uF, resistor:C-EUC0603
- added D1: IP4220CZ6, insole:IP4220CZ6
- added D2: CZRU52C4V7, insole:CZRU52C4V7
- added D3, D4: DB2G32600L1, insole:DB2G32600L1
- added D5, D6: (no value), resistor:R-EU_R0603
- added R11: 0, resistor:R-US_R0603
- added R26, R27: (no value), resistor:R-US_R0402
- R10: value 390k -> 75k
- R15: value 523k -> 110k
- R4: value 110k -> 523k
- R9: value 1.48M -> 374k
Connections:
- new net LDOIN: C17.1, R11.1, U8.VIN
- new net N$38: D5.2, R26.1
- new net N$39: D6.2, R27.1
- net +3V3: now also D1.IO4
- net 5V: now also D4.C
- net ADC7: now also D1.VP
- net D25: now also D1.IO1, D5.1
- net D27: now also D1.IO2, D6.1
- net D28: now also D1.IO3
- net GND: now also C7.2, D1.GND, D2.A, R26.2, R27.2
- net N$25: now also D3.A
- net N$26: now also D4.A
- net N$37: now also D3.C
- net OUT: now also C7.1, R11.2; no longer C17.1, U8.VIN
- net RECT: now also D2.C
Other:
- note added: "Zener diode"
- moved on the sheet: JP3
